File: Boards/INA186_BREAKOUT/INA186_Breakout.kicad_pcb (KiCad board)
At the start: 2 copper layers, 29.4 x 29.3 mm, 12 parts, among them U1 INA186

Commit message: Fixed File Structure
Fixed Branch organization and Fixed INA186 breakout edge cuts
Other:
- outline, holes or cut-outs redrawn
- board text added: "INA186 Dev Board Rev1"

Commit message: Research Library Updates
Copied over MRDT footprints, symbols, and 3D models to Research Library
Parts:
- added ?: , MRDT_Research:Debug_20mm, F.Cu at (65.1, 34.2)
