File: Boards/SerLCD_BREAKOUT/SerLCD_BREAKOUT/SerLCD_BREAKOUT.kicad_pcb (KiCad board)
At the start: 2 copper layers, 75 x 35 mm, 2 parts, among them U1 SerLCD, U2 Teensy4.1_DEV-16771

Commit message: Research Library Updates
Copied over MRDT footprints, symbols, and 3D models to Research Library
Parts:
- U1: footprint MRDT_Connectors:MOLEX_SL_03_Vertical -> MRDT_Research:MOLEX_SL_03_Vertical
- U2: value Teensy4.1_DEV-16771 -> Teensy4.1; footprint MRDT_Shields:MODULE_DEV-16771 -> MRDT_Research:Teensy 4.1
